File: 1_Hardware/magicwand2_1/magicwand2_1/magicwand2_1.kicad_sch (KiCad schematic)
At the start: 13 parts

Commit message: add lib folder
Parts:
- added U?: (no value), symbol Lib:LP2992IM5X-1.5/NOPB
- C?: value (none) -> 10nF
- C?: value (none) -> 100nF
- C?: value (none) -> 2.2nF
- R?: value (none) -> 10k
Other:
- moved on the sheet: C?, R?, U?

Commit message: schematic v1
Parts:
- added C? (x3): (no value), symbol Device:C
- added J?: (no value), symbol Connector:USB_C_Receptacle
- added Q? (x2): (no value), symbol Device:Q_NPN_BCE
- added R? (x6): (no value), symbol Device:R
- added U?: (no value), symbol Interface_USB:CP2102N-Axx-xQFN28
- U?: value (none) -> LP2992IM5X-1.5/NOPB; footprint (none) -> DBV0005A_N
Connections:
- net +5V is gone; now on net +3V3: C?.1, C?.1, C?.2, C?.2, R?.1, R?.1, R?.1, U?.1 (VDDA), U?.13 (VDD), U?.19 (VDD3P3_RTC), U?.3 (VDDA3P3), U?.37 (VDD3P3_CPU), U?.4 (VDDA3P3), U?.43 (VDDA), U?.46 (VDDA), U?.8 (VDDIO)
- net GND: now also U?.2 (GND), C?.1, C?.2, C?.2, J?.A1 (GND), J?.A12 (GND), J?.B1 (GND), J?.B12 (GND), J?.S1 (SHIELD), R?.2, R?.2, U?.29 (GND), U?.3 (GND)
- net GPIO0: now also Q?.2 (C)
- net VBUS: now reaches U?.1 (IN)
- net VBUS: now also U?.3 (ON_OFF_N), J?.A4 (VBUS), J?.A9 (VBUS), J?.B4 (VBUS), J?.B9 (VBUS), R?.2, U?.7 (VREGIN), U?.8 (VBUS)
- net at U?.4 (BYP): now also C?.2
- net +3V3: now reaches U?.5 (OUT)
- net +3V3: now also C?.1, C?.1
- new net: J?.B5 (CC2), R?.1
- new net: Q?.1 (B), R?.2 (x2)
- new net: R?.1, U?.26 (TXD)
- new net: R?.1, U?.9 (~{RST})
- new net: J?.A5 (CC1), R?.1
- new net CP_RX: U?.25 (RXD)
- new net CP_TX: R?.2
- new net DTR: Q?.3 (E), R?.1, U?.28 (~{DTR})
- new net EN: Q?.2 (C)
- new net RTS: Q?.3 (E), R?.1, U?.24 (~{RTS})
- new net USB-PWR-DM: J?.A7 (D-), J?.B7 (D-), U?.5 (D-)
- new net USB-PWR-DP: J?.A6 (D+), J?.B6 (D+), U?.4 (D+)
Other:
- note added: "Auto program circuit"
- moved on the sheet: U?

Commit message: correct 0811
Parts:
- C1: renamed from C?; value (none) -> 10nF
- C2: renamed from C?; value (none) -> 0.1uF
- C3: renamed from C?; value (none) -> 10uF
- J1: renamed from J?; value (none) -> USB_C_Receptacle
- Q1, Q2: renamed from Q?; value (none) -> Q_NPN_BCE
- R1, R2: renamed from R?; value (none) -> 5.1K
- R3, R4: renamed from R?; value (none) -> R
- R5: renamed from R?; value (none) -> 10K
- R6: renamed from R?; value (none) -> 200R
- U2: renamed from U?; value (none) -> CP2102N-Axx-xQFN28; footprint (none) -> Package_DFN_QFN:QFN-28-1EP_5x5mm_P0.5mm_EP3.35x3.35mm
- gave numbers to parts that had none: 14
Connections:
- net GPIO1 is gone; now on net CP_RX: U4.41 (U0TXD/IO1)
- net GPIO3 is gone; now on net CP_TX: U4.40 (U0RXD/IO3)
- net GPIO10: no longer names the net of U4.17 (IO14)
- net GPIO11: no longer names the net of U4.21 (IO15)
- net GPIO12: no longer names the net of U4.35 (IO18)
- net GPIO13: no longer names the net of U4.38 (IO19)
- net GPIO16: no longer names the net of U4.36 (IO23)
- net GPIO17: no longer names the net of U4.14 (IO25)
- net GPIO18: no longer names the net of U4.15 (IO26)
- net GPIO19: no longer names the net of U4.16 (IO27)
- net GPIO2: no longer names the net of U4.22 (IO2)
- net GPIO20: no longer names the net of U4.12 (IO32)
- net GPIO21: no longer names the net of U4.13 (IO33)
- net GPIO22: no longer names the net of U4.10 (IO34)
- net GPIO23: no longer names the net of U4.11 (IO35)
- net GPIO4: no longer names the net of U4.24 (IO4)
- net GPIO5: no longer names the net of U4.34 (IO5)
- net GPIO6: no longer names the net of U4.28 (SD2/IO9)
- net GPIO7: no longer names the net of U4.29 (SD3/IO10)
- net GPIO8: no longer names the net of U4.18 (IO12)
- net GPIO9: no longer names the net of U4.20 (IO13)
- net SENSOR_CAPN: no longer names the net of U4.7 (SENSOR_CAPN)
- net SENSOR_CAPP: no longer names the net of U4.6 (SENSOR_CAPP)
- net SENSOR_VN: no longer names the net of U4.8 (SENSOR_VN)
- net SENSOR_VP: no longer names the net of U4.5 (SENSOR_VP)
- no-connect marks 10 -> 60
